Commit message: Gazeboo and spawn fixed

File: furbo_description/urdf/furbo.urdf.xacro (robot description, xacro)
@@ -2,4 +2,31 @@
 <robot xmlns:xacro="http://www.ros.org/wiki/xacro"
        name="furbo">
+       <material name="blue">
+              <color rgba="0.2 0.4 0.9 1"/>
+          </material>
+          <material name="black">
+              <color rgba="0.1 0.1 0.1 1"/>
+          </material>
+          <material name="green">
+              <color rgba="0.0 0.8 0.0 1"/>
+          </material>
+          <material name="red">
+              <color rgba="0.9 0.1 0.1 1"/>
+          </material>
+          <material name="orange">
+              <color rgba="1.0 0.5 0.0 1"/>
+          </material>
+          <material name="yellow">
+              <color rgba="1.0 1.0 0.0 1"/>
+          </material>
+          <material name="gray">
+              <color rgba="0.6 0.6 0.6 1"/>
+       </material>
+       <link name="base_footprint"/>
+       <joint name="base_footprint_joint" type="fixed">
+              <parent link="base_footprint"/>
+              <child link="base_link"/>
+              <origin xyz="0 0 0.10"/>
+       </joint>
        <link name="base_link">
               <visual>
@@ -8,7 +35,5 @@
                             <box size="0.35 0.25 0.10"/>
                      </geometry>
-                     <material name="blue">
-                            <color rgba="0.2 0.4 0.9 1"/>
-                     </material>
+                     <material name="blue"/>
               </visual>
               <collision>
@@ -35,7 +60,5 @@
                       <cylinder radius="0.05" length="0.03"/>
                   </geometry>
-                  <material name="black">
-                      <color rgba="0.1 0.1 0.1 1"/>
-                  </material>
+                  <material name="black"/>
               </visual>
               <collision>
@@ -56,10 +79,191 @@
                       izz="0.0005"/>
               </inertial>
-          </link>
-          <joint name="left_wheel_joint" type="continuous">
+       </link>
+       <joint name="left_wheel_joint" type="continuous">
               <parent link="base_link"/>
               <child link="left_wheel"/>
-              <origin xyz="0 0.14 -0.05" rpy="0 0 0"/>
+              <origin xyz="0.03 0.14 -0.05" rpy="0 0 0"/>
               <axis xyz="0 1 0"/>
-          </joint>
+       </joint>
+       <link name="right_wheel">
+              <visual>
+                  <origin xyz="0 0 0" rpy="1.5708 0 0"/>
+                  <geometry>
+                      <cylinder radius="0.05" length="0.03"/>
+                  </geometry>
+                  <material name="black"/>
+              </visual>
+              <collision>
+                  <origin xyz="0 0 0" rpy="1.5708 0 0"/>
+                  <geometry>
+                      <cylinder radius="0.05" length="0.03"/>
+                  </geometry>
+              </collision>
+              <inertial>
+                  <mass value="0.3"/>
+                  <origin xyz="0 0 0"/>
+                  <inertia
+                      ixx="0.0005"
+                      ixy="0"
+                      ixz="0"
+                      iyy="0.0005"
+                      iyz="0"
+                      izz="0.0005"/>
+              </inertial>
+       </link>
+       <joint name="right_wheel_joint" type="continuous">
+              <parent link="base_link"/>
+              <child link="right_wheel"/>
+              <origin xyz="0.03 -0.14 -0.05" rpy="0 0 0"/>
+              <axis xyz="0 1 0"/>
+       </joint>
+       <link name="caster_wheel">
+              <visual>
+                  <origin xyz="0 0 0"/>
+                  <geometry>
+                      <sphere radius="0.05"/>
+                  </geometry>
+                  <material name="black"/>
+              </visual>
+              <collision>
+                  <origin xyz="0 0 0"/>
+                  <geometry>
+                      <sphere radius="0.05"/>
+                  </geometry>
+              </collision>
+              <inertial>
+                  <origin xyz="0 0 0"/>
+                  <mass value="0.1"/>
+                  <inertia
+                      ixx="0.0001"
+                      ixy="0"
+                      ixz="0"
+                      iyy="0.0001"
+                      iyz="0"
+                      izz="0.0001"/>
+              </inertial>
+       </link>
+       <joint name="caster_joint" type="fixed">
+              <parent link="base_link"/>
+              <child link="caster_wheel"/>
+              <origin xyz="-0.12 0 -0.05"/>
+       </joint>
+       <link name="lidar_link">
+              <visual>
+                  <origin xyz="0 0 0"/>
+                  <geometry>
+                      <cylinder radius="0.04" length="0.04"/>
+                  </geometry>
+                  <material name="green"/>
+              </visual>
+              <collision>
+                  <origin xyz="0 0 0"/>
+                  <geometry>
+                      <cylinder radius="0.04" length="0.04"/>
+                  </geometry>
+              </collision>
+              <inertial>
+                  <origin xyz="0 0 0"/>
+                  <mass value="0.2"/>
+                  <inertia
+                      ixx="0.0002"
+                      ixy="0"
+                      ixz="0"
+                      iyy="0.0002"
+                      iyz="0"
+                      izz="0.0002"/>
+              </inertial>
+       </link>
+       <joint name="lidar_joint" type="fixed">
+              <parent link="base_link"/>
+              <child link="lidar_link"/>
+              <origin xyz="0.00 0 0.09"/>
+       </joint>
+       <link name="imu_link">
+              <visual>
+                  <geometry>
+                      <box size="0.03 0.03 0.01"/>
+                  </geometry>
+                  <material name="orange"/>
+              </visual>
+              <collision>
+                  <geometry>
+                      <box size="0.03 0.03 0.01"/>
+                  </geometry>
+              </collision>
+              <inertial>
+                  <mass value="0.05"/>
+                  <origin xyz="0 0 0"/>
+                  <inertia
+                      ixx="0.00002"
+                      ixy="0"
+                      ixz="0"
+                      iyy="0.00002"
+                      iyz="0"
+                      izz="0.00002"/>
+              </inertial>
+       </link>
+       <joint name="imu_joint" type="fixed">
+              <parent link="base_link"/>
+              <child link="imu_link"/>
+              <origin xyz="0 0 0.03"/>
+       </joint>
+       <link name="camera_link">
+              <visual>
+                  <geometry>
+                      <box size="0.05 0.03 0.03"/>
+                  </geometry>
+                  <material name="red"/>
+              </visual>
+              <collision>
+                  <geometry>
+                      <box size="0.05 0.03 0.03"/>
+                  </geometry>
+              </collision>
+              <inertial>
+                  <mass value="0.10"/>
+                  <origin xyz="0 0 0"/>
+                  <inertia
+                      ixx="0.0001"
+                      ixy="0"
+                      ixz="0"
+                      iyy="0.0001"
+                      iyz="0"
+                      izz="0.0001"/>
+              </inertial>
+       </link>
+       <joint name="camera_joint" type="fixed">
+              <parent link="base_link"/>
+              <child link="camera_link"/>
+              <origin xyz="0.16 0 0.08"/>
+       </joint>
+       <link name="camera_optical_frame"/>
+       <joint name="camera_optical_joint" type="fixed">
+              <parent link="camera_link"/>
+              <child link="camera_optical_frame"/>
+              <origin xyz="0 0 0"
+                      rpy="-1.5708 0 -1.5708"/>
+       </joint>
+       <ros2_control name="furbo_system" type="system">
+            <hardware>
+                <plugin>gz_ros2_control/GazeboSimSystem</plugin>
+            </hardware>
+            <joint name="left_wheel_joint">
+                <command_interface name="velocity"/>
+                <state_interface name="position"/>
+                <state_interface name="velocity"/>
+            </joint>
+            <joint name="right_wheel_joint">
+                <command_interface name="velocity"/>
+                <state_interface name="position"/>
+                <state_interface name="velocity"/>
+            </joint>
+        </ros2_control>
+        <gazebo>
+            <plugin
+                filename="gz_ros2_control-system"
+                name="gz_ros2_control::GazeboSimROS2ControlPlugin">
+                <parameters>$(find furbo_description)/config/controllers.yaml</parameters>
+            </plugin>
+        </gazebo>
 </robot>

Commit message: Gazebo and ros2 timers fixed

File: furbo_description/urdf/furbo.urdf.xacro (robot description, xacro)
@@ -81,9 +81,11 @@
        </link>
        <joint name="left_wheel_joint" type="continuous">
-              <parent link="base_link"/>
-              <child link="left_wheel"/>
-              <origin xyz="0.03 0.14 -0.05" rpy="0 0 0"/>
-              <axis xyz="0 1 0"/>
-       </joint>
+            <parent link="base_link"/>
+            <child link="left_wheel"/>
+            <origin xyz="0.03 0.14 -0.05"/>
+            <axis xyz="0 1 0"/>
+            <limit effort="20" velocity="20"/>
+            <dynamics damping="0.0" friction="0.0"/>
+        </joint>
        <link name="right_wheel">
               <visual>
@@ -113,9 +115,11 @@
        </link>
        <joint name="right_wheel_joint" type="continuous">
-              <parent link="base_link"/>
-              <child link="right_wheel"/>
-              <origin xyz="0.03 -0.14 -0.05" rpy="0 0 0"/>
-              <axis xyz="0 1 0"/>
-       </joint>
+            <parent link="base_link"/>
+            <child link="right_wheel"/>
+            <origin xyz="0.03 -0.14 -0.05"/>
+            <axis xyz="0 1 0"/>
+            <limit effort="20" velocity="20"/>
+            <dynamics damping="0.0" friction="0.0"/>
+        </joint>
        <link name="caster_wheel">
               <visual>

Commit message: Camera added

File: furbo_description/urdf/furbo.urdf.xacro (robot description, xacro)
@@ -247,9 +247,4 @@
                   <material name="red"/>
               </visual>
-              <collision>
-                  <geometry>
-                      <box size="0.05 0.03 0.03"/>
-                  </geometry>
-              </collision>
               <inertial>
                   <mass value="0.10"/>
@@ -269,4 +264,23 @@
               <origin xyz="0.16 0 0.08"/>
        </joint>
+       <gazebo reference="camera_link">
+            <sensor name="camera" type="camera">
+                <pose>0.03 0 0 0 0 0</pose>
+                <topic>camera/image_raw</topic>
+                <update_rate>30</update_rate>
+                <camera>
+                    <horizontal_fov>1.047</horizontal_fov>
+                    <image>
+                        <width>640</width>
+                        <height>480</height>
+                    </image>
+                    <clip>
+                        <near>0.1</near>
+                        <far>100</far>
+                    </clip>
+                </camera>
+                <always_on>true</always_on>
+            </sensor>
+        </gazebo>
        <link name="camera_optical_frame"/>
        <joint name="camera_optical_joint" type="fixed">
