Commit message: SLAM implemented

File: furbo_description/urdf/furbo.urdf.xacro (robot description, xacro)
@@ -1,83 +1,83 @@
 <?xml version="1.0"?>
 <robot xmlns:xacro="http://www.ros.org/wiki/xacro"
-       name="furbo">
+    name="furbo">
        <material name="blue">
-              <color rgba="0.2 0.4 0.9 1"/>
-          </material>
-          <material name="black">
-              <color rgba="0.1 0.1 0.1 1"/>
-          </material>
-          <material name="green">
-              <color rgba="0.0 0.8 0.0 1"/>
-          </material>
-          <material name="red">
-              <color rgba="0.9 0.1 0.1 1"/>
-          </material>
-          <material name="orange">
-              <color rgba="1.0 0.5 0.0 1"/>
-          </material>
-          <material name="yellow">
-              <color rgba="1.0 1.0 0.0 1"/>
-          </material>
-          <material name="gray">
-              <color rgba="0.6 0.6 0.6 1"/>
+            <color rgba="0.2 0.4 0.9 1"/>
+        </material>
+        <material name="black">
+            <color rgba="0.1 0.1 0.1 1"/>
+        </material>
+        <material name="green">
+            <color rgba="0.0 0.8 0.0 1"/>
+        </material>
+        <material name="red">
+            <color rgba="0.9 0.1 0.1 1"/>
+        </material>
+        <material name="orange">
+            <color rgba="1.0 0.5 0.0 1"/>
+        </material>
+        <material name="yellow">
+            <color rgba="1.0 1.0 0.0 1"/>
+        </material>
+        <material name="gray">
+            <color rgba="0.6 0.6 0.6 1"/>
        </material>
        <link name="base_footprint"/>
        <joint name="base_footprint_joint" type="fixed">
-              <parent link="base_footprint"/>
-              <child link="base_link"/>
-              <origin xyz="0 0 0.10"/>
+            <parent link="base_footprint"/>
+            <child link="base_link"/>
+            <origin xyz="0 0 0.10"/>
        </joint>
        <link name="base_link">
-              <visual>
-                     <origin xyz="0 0 0" rpy="0 0 0"/>
-                     <geometry>
-                            <box size="0.35 0.25 0.10"/>
-                     </geometry>
-                     <material name="blue"/>
-              </visual>
-              <collision>
-                     <origin xyz="0 0 0" rpy="0 0 0"/>
-                     <geometry>
-                            <box size="0.35 0.25 0.10"/>
-                     </geometry>
-              </collision>
-              <inertial>
-                     <origin xyz="0 0 0" rpy="0 0 0"/>
-                     <mass value="5.0"/>
-                     <inertia ixx="0.0302"
-                     ixy="0.0"
-                     ixz="0.0"
-                     iyy="0.0552"
-                     iyz="0.0"
-                     izz="0.0771"/>
-              </inertial>
+            <visual>
+                <origin xyz="0 0 0" rpy="0 0 0"/>
+                <geometry>
+                <box size="0.35 0.25 0.10"/>
+                </geometry>
+                <material name="blue"/>
+            </visual>
+            <collision>
+                <origin xyz="0 0 0" rpy="0 0 0"/>
+                <geometry>
+                <box size="0.35 0.25 0.10"/>
+                </geometry>
+            </collision>
+            <inertial>
+                <origin xyz="0 0 0" rpy="0 0 0"/>
+                <mass value="5.0"/>
+                <inertia ixx="0.0302"
+                ixy="0.0"
+                ixz="0.0"
+                iyy="0.0552"
+                iyz="0.0"
+                izz="0.0771"/>
+            </inertial>
        </link>
        <link name="left_wheel">
-              <visual>
-                  <origin xyz="0 0 0" rpy="1.5708 0 0"/>
-                  <geometry>
-                      <cylinder radius="0.05" length="0.03"/>
-                  </geometry>
-                  <material name="black"/>
-              </visual>
-              <collision>
-                  <origin xyz="0 0 0" rpy="1.5708 0 0"/>
-                  <geometry>
-                      <cylinder radius="0.05" length="0.03"/>
-                  </geometry>
-              </collision>
-              <inertial>
-                  <mass value="0.3"/>
-                  <origin xyz="0 0 0"/>
-                  <inertia
-                      ixx="0.0005"
-                      ixy="0"
-                      ixz="0"
-                      iyy="0.0005"
-                      iyz="0"
-                      izz="0.0005"/>
-              </inertial>
-       </link>
+            <visual>
+                <origin xyz="0 0 0" rpy="1.5708 0 0"/>
+                <geometry>
+                    <cylinder radius="0.05" length="0.03"/>
+                </geometry>
+                <material name="black"/>
+            </visual>
+            <collision>
+                <origin xyz="0 0 0" rpy="1.5708 0 0"/>
+                <geometry>
+                <cylinder radius="0.05" length="0.03"/>
+                </geometry>
+            </collision>
+            <inertial>
+                <mass value="0.3"/>
+                <origin xyz="0 0 0"/>
+                <inertia
+                    ixx="0.0005"
+                    ixy="0"
+                    ixz="0"
+                    iyy="0.0005"
+                    iyz="0"
+                    izz="0.0005"/>
+            </inertial>
+        </link>
        <joint name="left_wheel_joint" type="continuous">
             <parent link="base_link"/>
@@ -88,29 +88,41 @@
             <dynamics damping="0.0" friction="0.0"/>
         </joint>
+        <gazebo reference="left_wheel">
+            <collision>
+                <surface>
+                    <friction>
+                        <ode>
+                            <mu>1.0</mu>
+                            <mu2>1.0</mu2>
+                        </ode>
+                    </friction>
+                </surface>
+            </collision>
+        </gazebo>
        <link name="right_wheel">
-              <visual>
-                  <origin xyz="0 0 0" rpy="1.5708 0 0"/>
-                  <geometry>
-                      <cylinder radius="0.05" length="0.03"/>
-                  </geometry>
-                  <material name="black"/>
-              </visual>
-              <collision>
-                  <origin xyz="0 0 0" rpy="1.5708 0 0"/>
-                  <geometry>
-                      <cylinder radius="0.05" length="0.03"/>
-                  </geometry>
-              </collision>
-              <inertial>
-                  <mass value="0.3"/>
-                  <origin xyz="0 0 0"/>
-                  <inertia
-                      ixx="0.0005"
-                      ixy="0"
-                      ixz="0"
-                      iyy="0.0005"
-                      iyz="0"
-                      izz="0.0005"/>
-              </inertial>
+            <visual>
+                <origin xyz="0 0 0" rpy="1.5708 0 0"/>
+                <geometry>
+                    <cylinder radius="0.05" length="0.03"/>
+                </geometry>
+                <material name="black"/>
+            </visual>
+            <collision>
+                <origin xyz="0 0 0" rpy="1.5708 0 0"/>
+                <geometry>
+                    <cylinder radius="0.05" length="0.03"/>
+                </geometry>
+            </collision>
+            <inertial>
+                <mass value="0.3"/>
+                <origin xyz="0 0 0"/>
+                <inertia
+                    ixx="0.0005"
+                    ixy="0"
+                    ixz="0"
+                    iyy="0.0005"
+                    iyz="0"
+                    izz="0.0005"/>
+            </inertial>
        </link>
        <joint name="right_wheel_joint" type="continuous">
@@ -122,65 +134,77 @@
             <dynamics damping="0.0" friction="0.0"/>
         </joint>
+        <gazebo reference="left_wheel">
+            <collision>
+                <surface>
+                    <friction>
+                        <ode>
+                            <mu>1.0</mu>
+                            <mu2>1.0</mu2>
+                        </ode>
+                    </friction>
+                </surface>
+            </collision>
+        </gazebo>
        <link name="caster_wheel">
-              <visual>
-                  <origin xyz="0 0 0"/>
-                  <geometry>
-                      <sphere radius="0.05"/>
-                  </geometry>
-                  <material name="black"/>
-              </visual>
-              <collision>
-                  <origin xyz="0 0 0"/>
-                  <geometry>
-                      <sphere radius="0.05"/>
-                  </geometry>
-              </collision>
-              <inertial>
-                  <origin xyz="0 0 0"/>
-                  <mass value="0.1"/>
-                  <inertia
-                      ixx="0.0001"
-                      ixy="0"
-                      ixz="0"
-                      iyy="0.0001"
-                      iyz="0"
-                      izz="0.0001"/>
-              </inertial>
+            <visual>
+                <origin xyz="0 0 0"/>
+                <geometry>
+                    <sphere radius="0.05"/>
+                </geometry>
+                <material name="black"/>
+            </visual>
+            <collision>
+                <origin xyz="0 0 0"/>
+                <geometry>
+                    <sphere radius="0.05"/>
+                </geometry>
+            </collision>
+            <inertial>
+                <origin xyz="0 0 0"/>
+                <mass value="0.1"/>
+                <inertia
+                    ixx="0.0001"
+                    ixy="0"
+                    ixz="0"
+                    iyy="0.0001"
+                    iyz="0"
+                    izz="0.0001"/>
+            </inertial>
        </link>
        <joint name="caster_joint" type="fixed">
-              <parent link="base_link"/>
-              <child link="caster_wheel"/>
-              <origin xyz="-0.12 0 -0.05"/>
+            <parent link="base_link"/>
+            <child link="caster_wheel"/>
+            <origin xyz="-0.12 0 -0.05"/>
        </joint>
        <link name="lidar_link">
-              <visual>
-                  <origin xyz="0 0 0"/>
-                  <geometry>
-                      <cylinder radius="0.04" length="0.04"/>
-                  </geometry>
-                  <material name="green"/>
-              </visual>
-              <collision>
-                  <origin xyz="0 0 0"/>
-                  <geometry>
-                      <cylinder radius="0.04" length="0.04"/>
-                  </geometry>
-              </collision>
-              <inertial>
-                  <origin xyz="0 0 0"/>
-                  <mass value="0.2"/>
-                  <inertia
-                      ixx="0.0002"
-                      ixy="0"
-                      ixz="0"
-                      iyy="0.0002"
-                      iyz="0"
-                      izz="0.0002"/>
-              </inertial>
+            <visual>
+                <origin xyz="0 0 0"/>
+                <geometry>
+                    <cylinder radius="0.04" length="0.04"/>
+                </geometry>
+                <material name="green"/>
+            </visual>
+            <collision>
+                <origin xyz="0 0 0"/>
+                <geometry>
+                    <cylinder radius="0.04" length="0.04"/>
+                </geometry>
+            </collision>
+            <inertial>
+                <origin xyz="0 0 0"/>
+                <mass value="0.2"/>
+                <inertia
+                    ixx="0.0002"
+                    ixy="0"
+                    ixz="0"
+                    iyy="0.0002"
+                    iyz="0"
+                    izz="0.0002"/>
+            </inertial>
        </link>
        <joint name="lidar_joint" type="fixed">
-              <parent link="base_link"/>
-              <child link="lidar_link"/>
-              <origin xyz="0.00 0 0.09"/>
+            <parent link="base_link"/>
+            <child link="lidar_link"/>
+            <origin xyz="0.00 0 0.09"/>
        </joint>
        <gazebo reference="lidar_link">
@@ -205,31 +229,31 @@
        </gazebo>
        <link name="imu_link">
-              <visual>
-                  <geometry>
-                      <box size="0.03 0.03 0.01"/>
-                  </geometry>
-                  <material name="orange"/>
-              </visual>
-              <collision>
-                  <geometry>
-                      <box size="0.03 0.03 0.01"/>
-                  </geometry>
-              </collision>
-              <inertial>
-                  <mass value="0.05"/>
-                  <origin xyz="0 0 0"/>
-                  <inertia
-                      ixx="0.00002"
-                      ixy="0"
-                      ixz="0"
-                      iyy="0.00002"
-                      iyz="0"
-                      izz="0.00002"/>
-              </inertial>
+            <visual>
+                <geometry>
+                    <box size="0.03 0.03 0.01"/>
+                </geometry>
+                <material name="orange"/>
+            </visual>
+            <collision>
+                <geometry>
+                    <box size="0.03 0.03 0.01"/>
+                </geometry>
+            </collision>
+            <inertial>
+                <mass value="0.05"/>
+                <origin xyz="0 0 0"/>
+                <inertia
+                    ixx="0.00002"
+                    ixy="0"
+                    ixz="0"
+                    iyy="0.00002"
+                    iyz="0"
+                    izz="0.00002"/>
+            </inertial>
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
Commit message: nav2 implemented

File: furbo_description/urdf/furbo.urdf.xacro (robot description, xacro)
@@ -2,5 +2,5 @@
 <robot xmlns:xacro="http://www.ros.org/wiki/xacro"
     name="furbo">
-       <material name="blue">
+        <material name="blue">
             <color rgba="0.2 0.4 0.9 1"/>
         </material>
@@ -22,5 +22,5 @@
         <material name="gray">
             <color rgba="0.6 0.6 0.6 1"/>
-       </material>
+        </material>
        <link name="base_footprint"/>
        <joint name="base_footprint_joint" type="fixed">
